Commit message: add friction and damping

File: urdf/ur_macro.xacro (robot description, xacro)
@@ -279,6 +279,9 @@
          <safety_controller soft_lower_limit="${shoulder_pan_lower_limit + safety_pos_margin}" soft_upper_limit="${shoulder_pan_upper_limit - safety_pos_margin}" k_position="${safety_k_position}" k_velocity="0.0"/>
       </xacro:if>
-      <dynamics damping="0" friction="0"/>
-    </joint>
+      <dynamics damping="0.7" friction="1.0"/>
+    </joint>
+    <gazebo reference="${prefix}shoulder_pan_joint">
+      <implicitSpringDamper>true</implicitSpringDamper>
+    </gazebo>
     <joint name="${tf_prefix}shoulder_lift_joint" type="revolute">
       <parent link="${tf_prefix}shoulder_link" />
@@ -291,6 +294,9 @@
          <safety_controller soft_lower_limit="${shoulder_lift_lower_limit + safety_pos_margin}" soft_upper_limit="${shoulder_lift_upper_limit - safety_pos_margin}" k_position="${safety_k_position}" k_velocity="0.0"/>
       </xacro:if>
-      <dynamics damping="0" friction="0"/>
-    </joint>
+      <dynamics damping="0.7" friction="1.0"/>
+    </joint>
+    <gazebo reference="${prefix}shoulder_lift_joint">
+      <implicitSpringDamper>true</implicitSpringDamper>
+    </gazebo>
     <joint name="${tf_prefix}elbow_joint" type="revolute">
       <parent link="${tf_prefix}upper_arm_link" />
@@ -303,6 +309,9 @@
          <safety_controller soft_lower_limit="${elbow_joint_lower_limit + safety_pos_margin}" soft_upper_limit="${elbow_joint_upper_limit - safety_pos_margin}" k_position="${safety_k_position}" k_velocity="0.0"/>
       </xacro:if>
-      <dynamics damping="0" friction="0"/>
-    </joint>
+      <dynamics damping="0.7" friction="1.0"/>
+    </joint>
+    <gazebo reference="${prefix}elbow_joint">
+      <implicitSpringDamper>true</implicitSpringDamper>
+    </gazebo>
     <joint name="${tf_prefix}wrist_1_joint" type="revolute">
       <parent link="${tf_prefix}forearm_link" />
@@ -315,6 +324,9 @@
          <safety_controller soft_lower_limit="${wrist_1_lower_limit + safety_pos_margin}" soft_upper_limit="${wrist_1_upper_limit - safety_pos_margin}" k_position="${safety_k_position}" k_velocity="0.0"/>
       </xacro:if>
-      <dynamics damping="0" friction="0"/>
-    </joint>
+      <dynamics damping="0.7" friction="1.0"/>
+    </joint>
+    <gazebo reference="${prefix}wrist_1_joint">
+      <implicitSpringDamper>true</implicitSpringDamper>
+    </gazebo>
     <joint name="${tf_prefix}wrist_2_joint" type="revolute">
       <parent link="${tf_prefix}wrist_1_link" />
@@ -327,6 +339,9 @@
          <safety_controller soft_lower_limit="${wrist_2_lower_limit + safety_pos_margin}" soft_upper_limit="${wrist_2_upper_limit - safety_pos_margin}" k_position="${safety_k_position}" k_velocity="0.0"/>
       </xacro:if>
-      <dynamics damping="0" friction="0"/>
-    </joint>
+      <dynamics damping="0.7" friction="1.0"/>
+    </joint>
+    <gazebo reference="${prefix}wrist_2_joint">
+      <implicitSpringDamper>true</implicitSpringDamper>
+    </gazebo>
     <joint name="${tf_prefix}wrist_3_joint" type="revolute">
       <parent link="${tf_prefix}wrist_2_link" />
@@ -339,6 +354,9 @@
          <safety_controller soft_lower_limit="${wrist_3_lower_limit + safety_pos_margin}" soft_upper_limit="${wrist_3_upper_limit - safety_pos_margin}" k_position="${safety_k_position}" k_velocity="0.0"/>
       </xacro:if>
-      <dynamics damping="0" friction="0"/>
-    </joint>
+      <dynamics damping="0.7" friction="1.0"/>
+    </joint>
+    <gazebo reference="${prefix}wrist_3_joint">
+      <implicitSpringDamper>true</implicitSpringDamper>
+    </gazebo>
     <link name="${tf_prefix}ft_frame"/>
     <joint name="${tf_prefix}wrist_3_link-ft_frame" type="fixed">
